File: RP2040 Board.kicad_pcb (KiCad board)
At the start: 2 copper layers, 31.5 x 30 mm, 28 parts, among them J1 USB_C_Receptacle_USB2.0, SW1 USB Boot Button, U1 RP2040, U2 ADP3338AKCZ-3.3, U3 W25Q128JVSIQ, X1 ABM8-272-T3

Commit message: Add files via upload
Parts:
- removed R6: Resistor, Resistor_SMD:R_0201_0603Metric
- removed SW1: USB Boot Button, Push Button:SW4_1825910-B_TEC
- removed U2: ADP3338AKCZ-3.3, PCM_4ms_Package_SOT:SOT89-3
- added R12: 1K, 1K Resistor:RC0402N_PAN, B.Cu at (137.5, 85.4)
- added U4: NCP1117LPST33T3G, Voltage:NCP1117, F.Cu at (150.0, 78.0)
- C1, C4: value Capacitor_NP -> 100nF; moved to B.Cu
- C10, C7: value Capacitor_NP -> 100nF; moved to F.Cu
- C11: value Capacitor_NP -> 1uF
- C12: value Capacitor_NP -> 10uF; moved to F.Cu
- C13: value Capacitor_NP -> 10uF; moved to B.Cu
- C14, C15: value Capacitor_10pF -> 15pF; moved to B.Cu
- C14_100n1, C2, C3, C5, C6, C9: value Capacitor_NP -> 100nF
- C8: value Capacitor_NP -> 1uF; moved to B.Cu
- R1: value Resistor -> 27Ω; footprint Resistor_SMD:R_0201_0603Metric -> PCM_Resistor_SMD_AKL:R_0402_1005Metric
- R2: value Resistor -> 27Ω; footprint Resistor_SMD:R_0201_0603Metric -> PCM_Resistor_SMD_AKL:R_0402_1005Metric; moved to B.Cu
- R3, R4: footprint Resistor_SMD:R_0201_0603Metric -> PCM_Resistor_SMD_AKL:R_0402_1005Metric
- R5: value Resistor -> 1K; footprint Resistor_SMD:R_0201_0603Metric -> 1K Resistor:RC0402N_PAN; moved to B.Cu
- U1, U3, X1: moved to B.Cu
- moved C1 16.0 mm to (131.8, 81.0)
- moved C7 15.9 mm to (136.0, 73.5), turned to 180 degrees
- moved C8 15.6 mm to (131.7, 72.5), turned to 0 degrees
- moved C14 12.5 mm to (145.5, 85.5)
- moved C3 12.3 mm to (136.3, 75.5)
- moved R5 12.0 mm to (144.0, 72.5), turned to 0 degrees
- moved C11 11.9 mm to (137.5, 77.8), turned to 90 degrees
- moved R2 7.77 mm to (137.5, 73.0)
- moved C2 7.43 mm to (135.7, 83.0)
- moved C13 7.28 mm to (146.0, 79.0), turned to 180 degrees
- moved C9 6.73 mm to (135.7, 81.0), turned to 0 degrees
- moved X1 6.49 mm to (142.1, 85.3)
- moved C6 6.35 mm to (140.9, 73.5)
- moved C14_100n1 4.30 mm to (136.2, 64.5), turned to 180 degrees
- moved C10 4.24 mm to (144.2, 74.0)
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Connections:
- C15 pad 2: Net-(U1-XOUT) -> Net-(C15-Pad2)
- R5 pad 2: 3v3 -> GPIO11
- U1 pad 11: unconnected-(U1-GPIO8-Pad11) -> GPIO08
- U1 pad 12: unconnected-(U1-GPIO9-Pad12) -> GPIO09
- U1 pad 13: unconnected-(U1-GPIO10-Pad13) -> GPIO10
- U1 pad 14: unconnected-(U1-GPIO11-Pad14) -> GPIO11
- U1 pad 15: unconnected-(U1-GPIO12-Pad15) -> GPIO12
- U1 pad 16: unconnected-(U1-GPIO13-Pad16) -> GPIO13
- U1 pad 17: unconnected-(U1-GPIO14-Pad17) -> GPIO14
- U1 pad 18: unconnected-(U1-GPIO15-Pad18) -> GPIO15
- U1 pad 2: unconnected-(U1-GPIO0-Pad2) -> GPIO00
- U1 pad 26: unconnected-(U1-RUN-Pad26) -> RUN
- U1 pad 27: unconnected-(U1-GPIO16-Pad27) -> GPIO16
- U1 pad 28: unconnected-(U1-GPIO17-Pad28) -> GPIO17
- U1 pad 29: unconnected-(U1-GPIO18-Pad29) -> GPIO18
- U1 pad 3: unconnected-(U1-GPIO1-Pad3) -> GPIO01
- U1 pad 30: unconnected-(U1-GPIO19-Pad30) -> GPIO19
- U1 pad 31: unconnected-(U1-GPIO20-Pad31) -> GPIO20
- U1 pad 32: unconnected-(U1-GPIO21-Pad32) -> GPIO21
- U1 pad 34: unconnected-(U1-GPIO22-Pad34) -> GPIO22
- U1 pad 4: unconnected-(U1-GPIO2-Pad4) -> GPIO02
- U1 pad 5: unconnected-(U1-GPIO3-Pad5) -> GPIO03
- U1 pad 6: unconnected-(U1-GPIO4-Pad6) -> GPIO04
- U1 pad 7: unconnected-(U1-GPIO5-Pad7) -> GPIO05
- U1 pad 8: unconnected-(U1-GPIO6-Pad8) -> GPIO06
- U1 pad 9: unconnected-(U1-GPIO7-Pad9) -> GPIO07
- X1 pad 3: Net-(U1-XOUT) -> Net-(C15-Pad2)
Routing:
- net Net-(J1-D--PadA7): track 12.1 -> 47.4 mm, vias 1 -> 0
- net Net-(J1-D+-PadA6): track 15.4 -> 47.9 mm, vias 2 -> 0
- net (no net): track 23.8 -> 0.00 mm, vias 1 -> 0
- net +1V1: track 28.8 -> 11.5 mm, vias 1 -> 3
- net GPIO11: track 0.00 -> 13.8 mm
- net Net-(R6-Pad1): track 13.5 -> 0.00 mm
- net Net-(U1-USB_DM): track 11.9 -> 2.17 mm, vias 2 -> 0
- net 3v3: track 139.4 -> 131.6 mm, vias 2 -> 10
- net Net-(U1-QSPI_SS): track 17.9 -> 10.6 mm, vias 1 -> 0
- net GND: track 30.5 -> 37.3 mm, vias 4 -> 5
- net unconnected-(U1-GND-Pad57): track 6.09 -> 0.00 mm, vias 1 -> 0
- net Net-(U1-USB_DP): track 7.32 -> 1.37 mm, vias 1 -> 0
- net unconnected-(U1-GPIO29_ADC3-Pad41): track 4.74 -> 0.00 mm
- net Net-(U1-QSPI_SD1): track 13.2 -> 8.58 mm
- net Net-(C15-Pad2): track 0.00 -> 4.31 mm
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- added copper zone on B.Cu, net GND
Other:
- board size 31.5 x 30 mm -> 25 x 27.5 mm
- board text added: "C7"
