File: RP2040 Board.kicad_sch (KiCad schematic)
At the start: 28 parts, among them J1 USB_C_Receptacle_USB2.0, SW1 USB Boot Button, U1 RP2040, U2 ADP3338AKCZ-3.3, U3 W25Q128JVSIQ, X1 ABM8-272-T3

Commit message: Add files via upload
Parts:
- removed R5, R6: Resistor, Resistor_SMD:R_0201_0603Metric, symbol PCM_SL_Resistors:Resistor
- removed SW1: USB Boot Button, Push Button:SW4_1825910-B_TEC, symbol PCM_SL_Devices:Push_Button_W12mm
- removed U2: ADP3338AKCZ-3.3, PCM_4ms_Package_SOT:SOT89-3, symbol PCM_Voltage_Regulator_AKL:ADP3338AKCZ-3.3
- added J2: Test Pins, symbol PCM_SL_Pin_Headers:PINHD_1x20_Female
- added R12, R5: 1K, 1K Resistor:RC0402N_PAN, symbol ERJ-2RKF1001X 1k Resistor:ERJ-2RKF1001X
- added U4: NCP1117LPST33T3G, Voltage:NCP1117, symbol PCM_4ms_Reference:NCP51460SN33
- C1, C10, C14_100n1, C2, C3, C4, C5, C6, C7, C9: value Capacitor_NP -> 100nF; Manufacturer (none) -> Samsung Electro-Mechanics; Part Number (none) -> CL10E104KC8VPNC
- C11, C8: value Capacitor_NP -> 1uF; Manufacturer (none) -> Samsung Electro-Mechanics; Part Number (none) -> CL10B105KP8NNNC
- C12, C13: value Capacitor_NP -> 10uF; Manufacturer (none) -> Samsung Electro-Mechanics; Part Number (none) -> CL10A106MQ8NNNC
- C14, C15: value Capacitor_10pF -> 15pF; Manufacturer (none) -> Würth Elektronik; Part Number (none) -> 885012006003
- J1: Manufacturer (none) -> G-Switch; Part Number (none) -> GT-USB-7010ASV
- R1, R2: value Resistor -> 27Ω; footprint Resistor_SMD:R_0201_0603Metric -> PCM_Resistor_SMD_AKL:R_0402_1005Metric; Manufacturer (none) -> Panasonic Electronic Components; Part Number (none) -> ERJ-2RKF27R0X
- R3, R4: footprint Resistor_SMD:R_0201_0603Metric -> PCM_Resistor_SMD_AKL:R_0402_1005Metric; Manufacturer (none) -> Panasonic Electronic Components; Part Number (none) -> ERA-2AEB512X
- U1: Manufacturer (none) -> Raspberry Pi; Part Number (none) -> SC0914(13)
- U3: Manufacturer (none) -> Winbond Electronics; Part Number (none) -> W25Q128JVSIQ
- X1: Manufacturer (none) -> Abracon LLC; Part Number (none) -> ABM8-272-T3
Connections:
- net 3v3: now also U4.2 (VO)
- net GND: now also U4.3 (GND)
- net at U1.56 (QSPI_SS), U3.1 (/CS): now also R5.1
- net at C12.1, J1.A4 (VBUS), J1.A9 (VBUS)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: now also U4.1 (VI)
- net at C15.2, X1.3: now also R12.2; no longer U1.21 (XOUT)
- net GPIO08: now reaches U1.11 (GPIO8)
- net GPIO09: now reaches U1.12 (GPIO9)
- net GPIO10: now reaches U1.13 (GPIO10)
- net GPIO11: now reaches U1.14 (GPIO11)
- net GPIO12: now reaches U1.15 (GPIO12)
- net GPIO13: now reaches U1.16 (GPIO13)
- net GPIO13: now also J2.3
- net GPIO14: now reaches U1.17 (GPIO14)
- net GPIO15: now reaches U1.18 (GPIO15)
- net GPIO00: now reaches U1.2 (GPIO0)
- net RUN: now reaches U1.26 (RUN)
- net RUN: now also J2.1
- net GPIO16: now reaches U1.27 (GPIO16)
- net GPIO16: now also J2.4
- net GPIO17: now reaches U1.28 (GPIO17)
- net GPIO17: now also J2.2
- net GPIO18: now reaches U1.29 (GPIO18)
- net GPIO01: now reaches U1.3 (GPIO1)
- net GPIO19: now reaches U1.30 (GPIO19)
- net GPIO20: now reaches U1.31 (GPIO20)
- net GPIO21: now reaches U1.32 (GPIO21)
- net GPIO22: now reaches U1.34 (GPIO22)
- net GPIO22: now also J2.6
- net GPIO02: now reaches U1.4 (GPIO2)
- net GPIO03: now reaches U1.5 (GPIO3)
- net GPIO04: now reaches U1.6 (GPIO4)
- net GPIO05: now reaches U1.7 (GPIO5)
- net GPIO06: now reaches U1.8 (GPIO6)
- net GPIO07: now reaches U1.9 (GPIO7)
- new net: R12.1, U1.21 (XOUT)
- new net SW6: R5.2
Other:
- moved on the sheet: C14
